File: eagle/buratino.sch (EAGLE design)
At the start: 57 parts, among them IC1 LTC3105MS, J1 Vcc-Vdd Tie, J2 Ext Battery, J4 Aux Batt, Q2 2n7002PW, U2 TPS78222, U4 ATMEGA256RFR2, U7 SWITCH, U8 LED-RGB, X1 16MHz, X2 32.768k, X3 AVR_JTAG, Y1 ANTENNA2SMD5

Commit message: pre-fab
Parts:
- added U$2: LOGO-OSHWSILKSCREEN, Pinoccio:LOGO-OSHWSILKSCREEN
- C16, C3, CFF: device Pinoccio:CAP0402-CAP -> Pinoccio:CAP0603-CAP
- RMPPC: device Pinoccio:RESISTOR0402-RES -> Pinoccio:RESISTOR0603-RES
- S1: value (none) -> BTN
- renumbered U$1 to PIR
Connections:
- net VCC: no longer JP-R.1
- net VIN: now also JP-R.1
Other:
- note added: "Copyright Buraitno 2014-2018"
- note removed: "Copyright Pinoccio 2012-2013"
Changed lines of the file:
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@@
 <part name="GND19" library="SparkFun" deviceset="GND" device=""/>
 <part name="GND23" library="SparkFun" deviceset="GND" device=""/>
-<part name="C3" library="Pinoccio" deviceset="CAP" device="0402-CAP" value="0.1uF"/>
+<part name="C3" library="Pinoccio" deviceset="CAP" device="0603-CAP" value="0.1uF"/>
 <part name="R22" library="Pinoccio" deviceset="RESISTOR" device="0603-RES" value="2K"/>
 <part name="R23" library="Pinoccio" deviceset="RESISTOR" device="0603-RES" value="2K"/>
@@
 <part name="TSL2561" library="@Sensors" deviceset="TSL2561" device="DFN" value="LUX"/>
 <part name="GND6" library="supply1" deviceset="GND" device=""/>
-<part name="C16" library="Pinoccio" deviceset="CAP" device="0402-CAP" value="0.1uF"/>
+<part name="C16" library="Pinoccio" deviceset="CAP" device="0603-CAP" value="0.1uF"/>
 <part name="L1" library="@Misc" deviceset="NR6045" device="T100M" value="10uH"/>
 <part name="SUPPLY1" library="supply2" deviceset="GND" device=""/>
@@
 <part name="SUPPLY6" library="supply2" deviceset="VDD" device=""/>
 <part name="CIN" library="Pinoccio" deviceset="CAP" device="0603-CAP" value="10uF"/>
-<part name="RMPPC" library="Pinoccio" deviceset="RESISTOR" device="0402-RES" value="30.1K"/>
+<part name="RMPPC" library="Pinoccio" deviceset="RESISTOR" device="0603-RES" value="30.1K"/>
 <part name="CAUX" library="Pinoccio" deviceset="CAP" device="0603-CAP" value="1.0uF"/>
 <part name="CLDO" library="Pinoccio" deviceset="CAP" device="0603-CAP" value="4.7uF"/>
-<part name="CFF" library="Pinoccio" deviceset="CAP" device="0402-CAP" value="22pF"/>
+<part name="CFF" library="Pinoccio" deviceset="CAP" device="0603-CAP" value="22pF"/>
 <part name="COUT" library="Pinoccio" deviceset="CAP" device="0603-CAP" value="1.0uF"/>
 <part name="R1" library="Pinoccio" deviceset="RESISTOR" device="0603-RES" value="1.37M"/>
@@
 <part name="J1" library="Pinoccio" deviceset="SOLDERJUMPER" device="NO" value="Vcc-Vdd Tie"/>
 <part name="J2" library="Pinoccio" deviceset="JUMPER-2" device="PTH" value="Ext Battery"/>
-<part name="S1" library="SparkFun-Electromechanical" deviceset="TAC_SWITCH" device="PTH"/>
+<part name="S1" library="SparkFun-Electromechanical" deviceset="TAC_SWITCH" device="PTH" value="BTN"/>
 <part name="R3" library="Pinoccio" deviceset="RESISTOR" device="0603-RES" value="10K"/>
 <part name="GND4" library="SparkFun" deviceset="GND" device=""/>
 <part name="SUPPLY7" library="supply2" deviceset="VDD" device=""/>
-<part name="U$1" library="620-Sensors" deviceset="IRS-B210ST01" device="R1"/>
+<part name="PIR" library="620-Sensors" deviceset="IRS-B210ST01" device="R1"/>
 <part name="SUPPLY8" library="supply2" deviceset="VDD" device=""/>
 <part name="GND7" library="SparkFun" deviceset="GND" device=""/>
 <part name="R4" library="Pinoccio" deviceset="RESISTOR" device="0603-RES" value="47K"/>
+<part name="U$2" library="Pinoccio" deviceset="LOGO-OSHW" device="SILKSCREEN"/>
 </parts>
 <sheets>
@@
 <text x="0" y="-0.127" size="0.0508" layer="21" font="vector">/Volumes/Data/Users/eric/Desktop/pinoccio-full-3-4in.bmp</text>
 <text x="0" y="-0.127" size="0.0508" layer="200" font="vector">/Volumes/Data/Users/eric/Desktop/pinoccio-full-3-4in.bmp</text>
-<text x="2.54" y="182.88" size="1.778" layer="95">Copyright Pinoccio 2012-2013</text>
+<text x="2.54" y="182.88" size="1.778" layer="95">Copyright Buraitno 2014-2018</text>
 <text x="2.54" y="180.34" size="1.778" layer="95">This documentation describes Open Hardware and is licensed under</text>
 <text x="2.54" y="177.8" size="1.778" layer="95">the CERN OHL v. 1.1. You may redistribute and modify this documentation </text>
@@
 </instance>
 <instance part="X3" gate="G$1" x="30.48" y="116.84"/>
-<instance part="SUPPLY3" gate="G$1" x="121.92" y="38.1"/>
+<instance part="SUPPLY3" gate="G$1" x="121.92" y="40.894"/>
 <instance part="J1" gate="1" x="121.92" y="30.988" rot="R90"/>
 <instance part="J2" gate="A" x="10.16" y="60.96" smashed="yes" rot="MR90">
@@
 <instance part="GND4" gate="1" x="124.46" y="63.5"/>
 <instance part="SUPPLY7" gate="G$1" x="154.94" y="73.66"/>
-<instance part="U$1" gate="G$1" x="119.38" y="83.82"/>
+<instance part="PIR" gate="G$1" x="119.38" y="83.82"/>
 <instance part="SUPPLY8" gate="G$1" x="101.6" y="93.98"/>
 <instance part="GND7" gate="1" x="114.3" y="76.2"/>
 <instance part="R4" gate="G$1" x="106.68" y="78.74" rot="R270"/>
+<instance part="U$2" gate="G$1" x="99.06" y="179.07"/>
 </instances>
 <busses>
@@
 </segment>
 <segment>
-<pinref part="U$1" gate="G$1" pin="GND"/>
+<pinref part="PIR" gate="G$1" pin="GND"/>
 <pinref part="GND7" gate="1" pin="GND"/>
 <wire x1="114.3" y1="81.28" x2="114.3" y2="78.74" width="0.1524" layer="91"/>
@@
 </segment>
 <segment>
-<pinref part="JP-R" gate="G$1" pin="1"/>
-<wire x1="236.22" y1="124.46" x2="223.52" y2="124.46" width="0.1524" layer="91"/>
-<label x="223.52" y="124.46" size="1.778" layer="95"/>
-</segment>
-<segment>
 <pinref part="JP-L" gate="G$1" pin="3"/>
 <wire x1="236.22" y1="172.72" x2="223.52" y2="172.72" width="0.1524" layer="91"/>
@@
 </segment>
 <segment>
-<pinref part="U$1" gate="G$1" pin="S"/>
+<pinref part="PIR" gate="G$1" pin="S"/>
 <pinref part="R4" gate="G$1" pin="1"/>
 <wire x1="101.6" y1="83.82" x2="106.68" y2="83.82" width="0.1524" layer="91"/>
@@
 <label x="86.36" y="27.178" size="1.778" layer="95" rot="R180"/>
 </segment>
+<segment>
+<pinref part="JP-R" gate="G$1" pin="1"/>
+<wire x1="236.22" y1="124.46" x2="223.52" y2="124.46" width="0.1524" layer="91"/>
+<label x="223.52" y="124.46" size="1.778" layer="95"/>
+</segment>
 </net>
 <net name="N$12" class="0">
@@
 <segment>
 <pinref part="SUPPLY3" gate="G$1" pin="VDD"/>
-<wire x1="121.92" y1="35.56" x2="121.92" y2="36.068" width="0.1524" layer="91"/>
+<wire x1="121.92" y1="38.354" x2="121.92" y2="36.068" width="0.1524" layer="91"/>
 <pinref part="J1" gate="1" pin="2"/>
 </segment>
@@
 <pinref part="SUPPLY8" gate="G$1" pin="VDD"/>
 <wire x1="101.6" y1="91.44" x2="101.6" y2="86.36" width="0.1524" layer="91"/>
-<pinref part="U$1" gate="G$1" pin="VIN"/>
+<pinref part="PIR" gate="G$1" pin="VIN"/>
 <wire x1="101.6" y1="86.36" x2="114.3" y2="86.36" width="0.1524" layer="91"/>
 </segment>

Commit message: add BOM, final tweaks
Parts:
- added J3: Vaux-Vcc Tie, Pinoccio:SOLDERJUMPERNO
- C12, C13, C14, C15: value 12pF -> 10pF
- C7, C8: device Pinoccio:CAP0402-CAP -> Pinoccio:CAP0603-CAP
- CIN: device Pinoccio:CAP0603-CAP -> Pinoccio:CAP0805
Connections:
- net VCC: now also J3.2
- net VCC-AE: now also J3.1
Other:
- moved on the sheet: C3, R5, U7
Changed lines of the file:
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@@
 <part name="GND1" library="SparkFun" deviceset="GND" device=""/>
 <part name="U4" library="Pinoccio" deviceset="ATMEGA128RFA1" device="" value="ATMEGA256RFR2"/>
-<part name="C7" library="Pinoccio" deviceset="CAP" device="0402-CAP" value="1.0uF"/>
-<part name="C8" library="Pinoccio" deviceset="CAP" device="0402-CAP" value="1.0uF"/>
-<part name="C13" library="Pinoccio" deviceset="CAP" device="0402-CAP" value="12pF"/>
-<part name="C12" library="Pinoccio" deviceset="CAP" device="0402-CAP" value="12pF"/>
-<part name="C15" library="Pinoccio" deviceset="CAP" device="0402-CAP" value="12pF"/>
-<part name="C14" library="Pinoccio" deviceset="CAP" device="0402-CAP" value="12pF"/>
+<part name="C7" library="Pinoccio" deviceset="CAP" device="0603-CAP" value="1.0uF"/>
+<part name="C8" library="Pinoccio" deviceset="CAP" device="0603-CAP" value="1.0uF"/>
+<part name="C13" library="Pinoccio" deviceset="CAP" device="0402-CAP" value="10pF"/>
+<part name="C12" library="Pinoccio" deviceset="CAP" device="0402-CAP" value="10pF"/>
+<part name="C15" library="Pinoccio" deviceset="CAP" device="0402-CAP" value="10pF"/>
+<part name="C14" library="Pinoccio" deviceset="CAP" device="0402-CAP" value="10pF"/>
 <part name="C9" library="Pinoccio" deviceset="CAP" device="0402-CAP" value="1.0pF"/>
 <part name="B1" library="Pinoccio" deviceset="BALUN" device="0805" value="BALUN"/>
@@
 <part name="S2" library="Pinoccio" deviceset="SWITCH-SPST" device="SMD2" value="SPST"/>
 <part name="SUPPLY6" library="supply2" deviceset="VDD" device=""/>
-<part name="CIN" library="Pinoccio" deviceset="CAP" device="0603-CAP" value="10uF"/>
+<part name="CIN" library="Pinoccio" deviceset="CAP" device="0805" value="10uF"/>
 <part name="RMPPC" library="Pinoccio" deviceset="RESISTOR" device="0603-RES" value="30.1K"/>
 <part name="CAUX" library="Pinoccio" deviceset="CAP" device="0603-CAP" value="1.0uF"/>
@@
 <part name="R4" library="Pinoccio" deviceset="RESISTOR" device="0603-RES" value="47K"/>
 <part name="U$2" library="Pinoccio" deviceset="LOGO-OSHW" device="SILKSCREEN"/>
+<part name="J3" library="Pinoccio" deviceset="SOLDERJUMPER" device="NO" value="Vaux-Vcc Tie"/>
+<part name="P+1" library="SparkFun" deviceset="VCC" device=""/>
 </parts>
 <sheets>
@@
 <attribute name="VALUE" x="137.922" y="47.498" size="1.778" layer="96" rot="MR0"/>
 </instance>
-<instance part="U7" gate="G$1" x="231.14" y="68.58" smashed="yes">
-<attribute name="NAME" x="223.52" y="67.31" size="1.778" layer="95"/>
+<instance part="U7" gate="G$1" x="218.44" y="63.5" smashed="yes">
+<attribute name="NAME" x="210.82" y="62.23" size="1.778" layer="95"/>
 </instance>
-<instance part="R5" gate="G$1" x="213.36" y="68.58" smashed="yes" rot="MR270">
-<attribute name="NAME" x="211.8614" y="69.85" size="1.778" layer="95" rot="MR270"/>
-<attribute name="VALUE" x="216.662" y="69.85" size="1.778" layer="96" rot="MR270"/>
-</instance>
-<instance part="GND19" gate="1" x="213.36" y="60.96"/>
-<instance part="GND23" gate="1" x="231.14" y="58.42"/>
-<instance part="C3" gate="G$1" x="238.76" y="66.04" smashed="yes">
-<attribute name="NAME" x="240.284" y="68.961" size="1.778" layer="95"/>
-<attribute name="VALUE" x="240.284" y="63.881" size="1.778" layer="96"/>
+<instance part="R5" gate="G$1" x="200.66" y="63.5" smashed="yes" rot="MR270">
+<attribute name="NAME" x="199.1614" y="64.77" size="1.778" layer="95" rot="MR270"/>
+<attribute name="VALUE" x="203.962" y="64.77" size="1.778" layer="96" rot="MR270"/>
+</instance>
+<instance part="GND19" gate="1" x="200.66" y="55.88"/>
+<instance part="GND23" gate="1" x="218.44" y="53.34"/>
+<instance part="C3" gate="G$1" x="226.06" y="60.96" smashed="yes">
+<attribute name="NAME" x="227.584" y="63.881" size="1.778" layer="95"/>
+<attribute name="VALUE" x="227.584" y="58.801" size="1.778" layer="96"/>
 </instance>
 <instance part="R22" gate="G$1" x="165.1" y="71.12" rot="R270"/>
@@
 <instance part="R4" gate="G$1" x="106.68" y="78.74" rot="R270"/>
 <instance part="U$2" gate="G$1" x="99.06" y="179.07"/>
+<instance part="J3" gate="1" x="233.68" y="71.12" rot="R90"/>
+<instance part="P+1" gate="1" x="233.68" y="76.2" smashed="yes">
+<attribute name="VALUE" x="225.806" y="77.47" size="1.778" layer="96"/>
+</instance>
 </instances>
 <busses>
@@
 <pinref part="U7" gate="G$1" pin="GND"/>
 <pinref part="GND23" gate="1" pin="GND"/>
-<wire x1="231.14" y1="60.96" x2="231.14" y2="63.5" width="0.1524" layer="91"/>
+<wire x1="218.44" y1="55.88" x2="218.44" y2="58.42" width="0.1524" layer="91"/>
 <pinref part="C3" gate="G$1" pin="2"/>
-<wire x1="231.14" y1="63.5" x2="231.14" y2="66.04" width="0.1524" layer="91"/>
-<wire x1="238.76" y1="63.5" x2="231.14" y2="63.5" width="0.1524" layer="91"/>
-<junction x="231.14" y="63.5"/>
+<wire x1="218.44" y1="58.42" x2="218.44" y2="60.96" width="0.1524" layer="91"/>
+<wire x1="226.06" y1="58.42" x2="218.44" y2="58.42" width="0.1524" layer="91"/>
+<junction x="218.44" y="58.42"/>
 </segment>
 <segment>
@@
 <segment>
 <pinref part="U7" gate="G$1" pin="IN"/>
-<wire x1="220.98" y1="71.12" x2="226.06" y2="71.12" width="0.1524" layer="91"/>
-<label x="220.98" y="71.12" size="1.778" layer="95"/>
+<wire x1="208.28" y1="66.04" x2="213.36" y2="66.04" width="0.1524" layer="91"/>
+<label x="208.28" y="66.04" size="1.778" layer="95"/>
 </segment>
 <segment>
@@
 <label x="223.52" y="172.72" size="1.778" layer="95"/>
 </segment>
+<segment>
+<pinref part="J3" gate="1" pin="2"/>
+<pinref part="P+1" gate="1" pin="VCC"/>
+</segment>
 </net>
 <net name="MOSI" class="0">
@@
 <segment>
 <pinref part="U7" gate="G$1" pin="OUT"/>
-<wire x1="233.68" y1="71.12" x2="238.76" y2="71.12" width="0.1524" layer="91"/>
-<label x="236.22" y="71.12" size="1.778" layer="95"/>
+<wire x1="220.98" y1="66.04" x2="226.06" y2="66.04" width="0.1524" layer="91"/>
+<label x="223.52" y="66.04" size="1.778" layer="95"/>
 <pinref part="C3" gate="G$1" pin="1"/>
-<wire x1="238.76" y1="71.12" x2="246.38" y2="71.12" width="0.1524" layer="91"/>
-<junction x="238.76" y="71.12"/>
+<wire x1="226.06" y1="66.04" x2="233.68" y2="66.04" width="0.1524" layer="91"/>
+<junction x="226.06" y="66.04"/>
+<pinref part="J3" gate="1" pin="1"/>
 </segment>
 <segment>
@@
 <segment>
 <pinref part="U7" gate="G$1" pin="ON"/>
-<wire x1="231.14" y1="76.2" x2="213.36" y2="76.2" width="0.1524" layer="91"/>
+<wire x1="218.44" y1="71.12" x2="200.66" y2="71.12" width="0.1524" layer="91"/>
 <pinref part="R5" gate="G$1" pin="1"/>
-<wire x1="213.36" y1="73.66" x2="213.36" y2="76.2" width="0.1524" layer="91"/>
-<wire x1="213.36" y1="76.2" x2="205.74" y2="76.2" width="0.1524" layer="91"/>
-<junction x="213.36" y="76.2"/>
-<label x="205.74" y="76.2" size="1.778" layer="95"/>
+<wire x1="200.66" y1="68.58" x2="200.66" y2="71.12" width="0.1524" layer="91"/>
+<wire x1="200.66" y1="71.12" x2="193.04" y2="71.12" width="0.1524" layer="91"/>
+<junction x="200.66" y="71.12"/>
+<label x="193.04" y="71.12" size="1.778" layer="95"/>
 </segment>
 <segment>
